File: Hardware/Schematics, PCB layouts/OscilloBP Monitor/OscilloBP Monitor.kicad_pcb (KiCad board)
At the start: 2 copper layers, 3 parts, among them U1 ZC323000

Commit message: Tìm linh kiện upload
Parts:
- added C2: 100nF, Capacitor_SMD:C_0603_1608Metric, F.Cu at (77.7, 120.5)
- added C3: 10uF, Capacitor_Tantalum_SMD:CP_EIA-1608-08_AVX-J_HandSolder, F.Cu at (68.2, 132.5)
- added L1: 22uH, CDRH104:CDRH104, F.Cu at (58.5, 118.5)
- added Q1: BSS138, Package_TO_SOT_SMD:SOT-23, F.Cu at (54.6, 133.0)
- added U2: MT3608, Package_TO_SOT_SMD:SOT-23-6, F.Cu at (39.9, 128.4)
- C1: footprint Capacitor_THT:CP_Radial_D8.0mm_P5.00mm -> Capacitor_THT:CP_Radial_D16.0mm_P7.50mm

Commit message: Thêm schematic.pdf
Parts:
- removed C1: 1000uF - 16V, Capacitor_THT:CP_Radial_D16.0mm_P7.50mm
- removed C2: 100nF, Capacitor_SMD:C_0603_1608Metric
- removed C3: 10uF, Capacitor_Tantalum_SMD:CP_EIA-1608-08_AVX-J_HandSolder
- removed D1: 1N5819-G, 1N5819G:DIOAD1405W75L465D235
- added BT101: Battery_Cell, Battery1:1x18650, F.Cu at (56.0, 30.5)
- added C101: 22uF, Capacitor_SMD:C_1206_3216Metric_Pad1.33x1.80mm_HandSolder, F.Cu at (79.4, 102.7)
- added C102: 22uF, Capacitor_SMD:C_1206_3216Metric_Pad1.33x1.80mm_HandSolder, F.Cu at (79.4, 99.3)
- added C201: 1000uF - 16tV, Capacitor_THT:CP_Radial_D16.0mm_P7.50mm, F.Cu at (77.0, 134.0)
- added C501: 1µF, Capacitor_SMD:C_1206_3216Metric_Pad1.33x1.80mm_HandSolder, F.Cu at (190.9, 54.5)
- added C502: 1µF, Capacitor_SMD:C_1206_3216Metric_Pad1.33x1.80mm_HandSolder, F.Cu at (236.3, 48.8)
- added C601: 10nF, Capacitor_SMD:C_1206_3216Metric_Pad1.33x1.80mm_HandSolder, F.Cu at (236.3, 52.1)
- added C602: 1µF, Capacitor_SMD:C_1206_3216Metric_Pad1.33x1.80mm_HandSolder, F.Cu at (236.3, 55.5)
- added C603: 470pF, Capacitor_SMD:C_1206_3216Metric_Pad1.33x1.80mm_HandSolder, F.Cu at (236.3, 58.9)
- added D101: SS34, Diode_SMD:D_SMA, F.Cu at (80.7, 95.4)
- added D201: 1N5819, Diode_THT:D_DO-41_SOD81_P10.16mm_Horizontal, F.Cu at (157.8, 109.8)
- added D202: 1N5819, Diode_THT:D_DO-41_SOD81_P10.16mm_Horizontal, F.Cu at (157.8, 114.0)
- added D401: LED_RED, LED_THT:LED_D3.0mm, F.Cu at (72.4, 89.5)
- added D402: LED_GREEN, LED_THT:LED_D3.0mm, F.Cu at (72.4, 95.0)
- added D403: LED_YELLOW, LED_THT:LED_D3.0mm, F.Cu at (72.4, 100.4)
- added FB601: CBG201209U252T, Inductor_SMD:L_0805_2012Metric_Pad1.05x1.20mm_HandSolder, F.Cu at (190.3, 57.5)
- added H1: MountingHole_Pad, MountingHole_3.2mm_M3_Pad_Via_Silk:MountingHole_3.2mm_M3_Pad_Via_Silk, F.Cu at (70.0, 58.0)
- added H2: MountingHole_Pad, MountingHole_3.2mm_M3_Pad_Via_Silk:MountingHole_3.2mm_M3_Pad_Via_Silk, F.Cu at (83.3, 59.3)
- added H3: MountingHole_Pad, MountingHole_3.2mm_M3_Pad_Via_Silk:MountingHole_3.2mm_M3_Pad_Via_Silk, F.Cu at (100.1, 62.0)
- added H4: MountingHole_Pad, MountingHole_3.2mm_M3_Pad_Via_Silk:MountingHole_3.2mm_M3_Pad_Via_Silk, F.Cu at (114.3, 64.7)
- added J201: Terminal_01x04, TerminalBlock_KF:TerminalBlock_KF_1x04_P7.62mm_Vertical, F.Cu at (72.8, 84.7)
- added Q201: AO3400A, AO3400A:SOT95P280X125-3N, F.Cu at (109.7, 39.0)
- added Q202: AO3400A, AO3400A:SOT95P280X125-3N, F.Cu at (172.9, 110.0)
- added Q302: BSS138, Package_TO_SOT_SMD:SOT-23, F.Cu at (175.2, 96.6)
- added R101: 2.2K, Resistor_SMD:R_1206_3216Metric_Pad1.30x1.75mm_HandSolder, F.Cu at (164.4, 99.3)
- added R201: 100R, Resistor_SMD:R_1206_3216Metric_Pad1.30x1.75mm_HandSolder, F.Cu at (158.8, 102.7)
- added R202: 10k, Resistor_SMD:R_1206_3216Metric_Pad1.30x1.75mm_HandSolder, F.Cu at (158.8, 96.0)
- added R203: 100R, Resistor_SMD:R_1206_3216Metric_Pad1.30x1.75mm_HandSolder, F.Cu at (158.8, 106.0)
- added R204: 10k, Resistor_SMD:R_1206_3216Metric_Pad1.30x1.75mm_HandSolder, F.Cu at (158.8, 99.3)
- added R301: 10k, Resistor_SMD:R_1206_3216Metric_Pad1.30x1.75mm_HandSolder, F.Cu at (164.4, 102.7)
- added R302: 10k, Resistor_SMD:R_1206_3216Metric_Pad1.30x1.75mm_HandSolder, F.Cu at (236.3, 68.2)
- added R303: 10k, Resistor_SMD:R_1206_3216Metric_Pad1.30x1.75mm_HandSolder, F.Cu at (164.4, 96.0)
- added R304: 10k, Resistor_SMD:R_1206_3216Metric_Pad1.30x1.75mm_HandSolder, F.Cu at (164.4, 106.0)
- added R401: 220R, Resistor_SMD:R_1206_3216Metric_Pad1.30x1.75mm_HandSolder, F.Cu at (170.0, 99.3)
- added R402: 220R, Resistor_SMD:R_1206_3216Metric_Pad1.30x1.75mm_HandSolder, F.Cu at (170.0, 102.7)
- added R403: 220R, Resistor_SMD:R_1206_3216Metric_Pad1.30x1.75mm_HandSolder, F.Cu at (170.0, 106.0)
- added R501: 1K, Resistor_SMD:R_1206_3216Metric_Pad1.30x1.75mm_HandSolder, F.Cu at (236.3, 71.5)
- added R502: 10K, Resistor_SMD:R_1206_3216Metric_Pad1.30x1.75mm_HandSolder, F.Cu at (185.0, 107.0)
- added RV101: 100K, Potentiometer_THT:Potentiometer_Bourns_3296W_Vertical, F.Cu at (84.7, 89.9)
- added SW_HIGH401: SW_Push, Button_Switch_THT:SW_SPST_Omron_B3F-40xx, F.Cu at (219.0, 52.4)
- added SW_START401: SW_Push, Button_Switch_THT:SW_SPST_Omron_B3F-40xx, F.Cu at (219.0, 68.0)
- added SW_STOP401: SW_Push, Button_Switch_THT:SW_SPST_Omron_B3F-40xx, F.Cu at (219.0, 83.5)
- added U101: TP4056, TP4056_Module:TP4056_Module, F.Cu at (30.3, 47.7)
- added U501: ADS1115IDGST, ADS1115:ADS1115_MSOP10, F.Cu at (197.0, 113.5)
- added U601: MPXV5050GP, MPXV5050GP:SOIC127P600X175-8N, F.Cu at (237.4, 63.5)
- renumbered L1 to L101, Q1 to Q301, U2 to U102, U1 to U401
Connections:
- L101 pad 1: unconnected-(L1-Pad1) -> +3.7V
- L101 pad 2: unconnected-(L1-Pad2) -> Net-(D101-A)
- Q301 pad 1: unconnected-(Q1-G-Pad1) -> +3.3V
- Q301 pad 2: unconnected-(Q1-S-Pad2) -> /SDA_STM32
- Q301 pad 3: unconnected-(Q1-D-Pad3) -> /SDA_ADC
- U102 pad 1: unconnected-(U2-SW-Pad1) -> Net-(D101-A)
- U102 pad 2: unconnected-(U2-GND-Pad2) -> DGND
- U102 pad 3: unconnected-(U2-FB-Pad3) -> Net-(U102-FB)
- U102 pad 4: unconnected-(U2-EN-Pad4) -> +3.7V
- U102 pad 5: unconnected-(U2-IN-Pad5) -> +3.7V
- U401 pad 10: unconnected-(U1-A5-Pad10) -> Net-(U401-A5)
- U401 pad 11: unconnected-(U1-A6-Pad11) -> Net-(U401-A6)
- U401 pad 12: unconnected-(U1-A7-Pad12) -> Net-(U401-A7)
- U401 pad 18: 3.3 -> +3.3V
- U401 pad 19: G -> DGND
- U401 pad 20: G -> DGND
- U401 pad 22: unconnected-(U1-B13-Pad22) -> Net-(U401-B13)
- U401 pad 23: unconnected-(U1-B14-Pad23) -> Net-(U401-B14)
- U401 pad 24: unconnected-(U1-B15-Pad24) -> Net-(U401-B15)
- U401 pad 34: unconnected-(U1-B6-Pad34) -> /SCL_STM32
- U401 pad 35: unconnected-(U1-B7-Pad35) -> /SDA_STM32
- U401 pad 38: unconnected-(U1-5V-Pad38) -> +5V
- U401 pad 39: G -> DGND
- U401 pad 40: 3.3 -> +3.3V
- U401 pad 5: unconnected-(U1-A0-Pad5) -> /PWM_Motor
- U401 pad 6: unconnected-(U1-A1-Pad6) -> /PWM_Valve
